File: LargeHeader/Header.brd (EAGLE design)
At the start: 35.9 x 52.1 mm, 4 parts

Commit message: Shifted text to not be blocked by header
Other:
- board size 35.9 x 52.1 mm -> 37.1 x 52.1 mm
Changed lines of the file:
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@@
 <setting verticaltext="up"/>
 </settings>
-<grid distance="0.025" unitdist="inch" unit="inch" style="lines" multiple="1" display="yes" altdistance="0.0125" altunitdist="inch" altunit="inch"/>
+<grid distance="25" unitdist="mil" unit="mil" style="lines" multiple="1" display="yes" altdistance="0.0125" altunitdist="inch" altunit="inch"/>
 <layers>
 <layer number="1" name="Top" color="4" fill="1" visible="yes" active="yes"/>
@@
 <board>
 <plain>
-<wire x1="0" y1="0" x2="35.865" y2="0" width="0" layer="20"/>
-<wire x1="35.865" y1="0" x2="35.865" y2="52.06" width="0" layer="20"/>
-<wire x1="35.865" y1="52.06" x2="0" y2="52.06" width="0" layer="20"/>
+<wire x1="0" y1="0" x2="37.135" y2="0" width="0" layer="20"/>
+<wire x1="37.135" y1="0" x2="37.135" y2="52.06" width="0" layer="20"/>
+<wire x1="37.135" y1="52.06" x2="0" y2="52.06" width="0" layer="20"/>
 <wire x1="0" y1="52.06" x2="0" y2="0" width="0" layer="20"/>
-<text x="27.305" y="34.29" size="1.27" layer="21">3.3V</text>
-<text x="27.305" y="31.75" size="1.27" layer="21">2/SDA</text>
-<text x="27.305" y="29.21" size="1.27" layer="21">3/SCL</text>
-<text x="27.305" y="26.67" size="1.27" layer="21">4</text>
-<text x="27.305" y="24.13" size="1.27" layer="21">GND</text>
-<text x="27.305" y="21.59" size="1.27" layer="21">17/RTS</text>
-<text x="27.305" y="19.05" size="1.27" layer="21">27</text>
-<text x="27.305" y="16.51" size="1.27" layer="21">22</text>
-<text x="27.305" y="13.97" size="1.27" layer="21">3.3V</text>
-<text x="27.305" y="11.43" size="1.27" layer="21">10/MOSI</text>
-<text x="27.305" y="8.89" size="1.27" layer="21">9/MISO</text>
-<text x="27.305" y="6.35" size="1.27" layer="21">11/CLK</text>
-<text x="27.305" y="3.81" size="1.27" layer="21">GND</text>
-<text x="22.225" y="35.56" size="1.27" layer="21" align="top-right">5V</text>
-<text x="22.225" y="33.02" size="1.27" layer="21" align="top-right">5V</text>
-<text x="22.225" y="27.94" size="1.27" layer="21" align="top-right">14/TX</text>
-<text x="22.225" y="25.4" size="1.27" layer="21" align="top-right">15/RX</text>
-<text x="22.225" y="22.86" size="1.27" layer="21" align="top-right">18</text>
-<text x="22.225" y="20.32" size="1.27" layer="21" align="top-right">GND</text>
-<text x="22.225" y="17.78" size="1.27" layer="21" align="top-right">23</text>
-<text x="22.225" y="15.24" size="1.27" layer="21" align="top-right">24</text>
-<text x="22.225" y="12.7" size="1.27" layer="21" align="top-right">GND</text>
-<text x="22.225" y="10.16" size="1.27" layer="21" align="top-right">25</text>
-<text x="22.225" y="7.62" size="1.27" layer="21" align="top-right">8/CE0</text>
-<text x="22.225" y="5.08" size="1.27" layer="21" align="top-right">7/CE1</text>
-<text x="22.225" y="30.48" size="1.27" layer="21" align="top-right">GND</text>
+<text x="28.575" y="34.29" size="1.27" layer="21">3.3V</text>
+<text x="28.575" y="31.75" size="1.27" layer="21">2/SDA</text>
+<text x="28.575" y="29.21" size="1.27" layer="21">3/SCL</text>
+<text x="28.575" y="26.67" size="1.27" layer="21">4</text>
+<text x="28.575" y="24.13" size="1.27" layer="21">GND</text>
+<text x="28.575" y="21.59" size="1.27" layer="21">17/RTS</text>
+<text x="28.575" y="19.05" size="1.27" layer="21">27</text>
+<text x="28.575" y="16.51" size="1.27" layer="21">22</text>
+<text x="28.575" y="13.97" size="1.27" layer="21">3.3V</text>
+<text x="28.575" y="11.43" size="1.27" layer="21">10/MOSI</text>
+<text x="28.575" y="8.89" size="1.27" layer="21">9/MISO</text>
+<text x="28.575" y="6.35" size="1.27" layer="21">11/CLK</text>
+<text x="28.575" y="3.81" size="1.27" layer="21">GND</text>
+<text x="21.59" y="35.56" size="1.27" layer="21" align="top-right">5V</text>
+<text x="21.59" y="32.385" size="1.27" layer="21" align="top-right">5V</text>
+<text x="21.59" y="27.94" size="1.27" layer="21" align="top-right">14/TX</text>
+<text x="21.59" y="25.4" size="1.27" layer="21" align="top-right">15/RX</text>
+<text x="21.59" y="22.86" size="1.27" layer="21" align="top-right">18</text>
+<text x="21.59" y="20.32" size="1.27" layer="21" align="top-right">GND</text>
+<text x="21.59" y="17.78" size="1.27" layer="21" align="top-right">23</text>
+<text x="21.59" y="15.24" size="1.27" layer="21" align="top-right">24</text>
+<text x="21.59" y="12.7" size="1.27" layer="21" align="top-right">GND</text>
+<text x="21.59" y="10.16" size="1.27" layer="21" align="top-right">25</text>
+<text x="21.59" y="7.62" size="1.27" layer="21" align="top-right">8/CE0</text>
+<text x="21.59" y="5.08" size="1.27" layer="21" align="top-right">7/CE1</text>
+<text x="21.59" y="30.48" size="1.27" layer="21" align="top-right">GND</text>
 <circle x="11.43" y="41.91" radius="3.862553125" width="0.4064" layer="49"/>
 <circle x="11.43" y="8.255" radius="2.54" width="0.4064" layer="49"/>
@@
 The double circles are on the reference layer and
 will not be printed on the PCB</text>
-<text x="27.305" y="41.91" size="1.27" layer="21">GND</text>
-<text x="27.305" y="44.45" size="1.27" layer="21">SPK</text>
-<text x="22.225" y="43.18" size="1.27" layer="21" align="top-right">AUDIO</text>
-<text x="22.225" y="45.72" size="1.27" layer="21" align="top-right">SPK</text>
+<text x="28.575" y="41.91" size="1.27" layer="21">GND</text>
+<text x="28.575" y="44.45" size="1.27" layer="21">SPK</text>
+<text x="21.59" y="43.18" size="1.27" layer="21" align="top-right">AUDIO</text>
+<text x="21.59" y="45.72" size="1.27" layer="21" align="top-right">SPK</text>
 <polygon width="0.4064" layer="41">
 <vertex x="11.43" y="45.72" curve="90"/>
@@
 <text x="28.575" y="49.53" size="1.778" layer="21">J3</text>
 <text x="5.715" y="49.53" size="1.778" layer="21">J4</text>
-<text x="27.305" y="39.37" size="1.27" layer="21">EXT</text>
-<text x="31.4325" y="39.37" size="1.27" layer="21">GND</text>
-<text x="27.305" y="36.83" size="1.27" layer="21">EXT</text>
-<text x="31.4325" y="36.83" size="1.27" layer="21">GND</text>
-<text x="22.225" y="40.64" size="1.27" layer="21" align="top-right">5V</text>
-<text x="22.225" y="38.1" size="1.27" layer="21" align="top-right">3.3V</text>
-<text x="19.3675" y="40.64" size="1.27" layer="21" align="top-right">EXT</text>
-<text x="17.78" y="38.1" size="1.27" layer="21" align="top-right">EXT</text>
+<text x="28.575" y="39.37" size="1.27" layer="21">EXT</text>
+<text x="32.7025" y="39.37" size="1.27" layer="21">GND</text>
+<text x="28.575" y="36.83" size="1.27" layer="21">EXT</text>
+<text x="32.7025" y="36.83" size="1.27" layer="21">GND</text>
+<text x="21.59" y="40.64" size="1.27" layer="21" align="top-right">5V</text>
+<text x="21.59" y="38.1" size="1.27" layer="21" align="top-right">3.3V</text>
+<text x="18.7325" y="40.64" size="1.27" layer="21" align="top-right">EXT</text>
+<text x="16.51" y="38.1" size="1.27" layer="21" align="top-right">EXT</text>
 </plain>
 <attributes>
